File: cad/top-octave.kicad_sch (KiCad schematic)
At the start: 7 parts, among them Q1 Q_NJFET_DGS, U9 ATtiny4-TS

Commit message: Update schematic
Parts:
- removed C?: 1u, symbol Device:C_Polarized_Small_US
- removed C?: 10u, symbol Device:C_Polarized_Small_US
- removed U?: AMS1117-5.0, Package_TO_SOT_SMD:SOT-223-3_TabPin2, symbol Regulator_Linear:AMS1117-5.0
- added C1: 39p, symbol Device:C_Small
- added C10, C17: 22u, symbol Device:C_Polarized_Small_US
- added C11, C12, C13, C14, C15, C16, C2, C4, C5, C7, C8, C9: 100n, Capacitor_SMD:C_1206_3216Metric_Pad1.42x1.75mm_HandSolder, symbol Device:C_Small
- added C3: 68p, symbol Device:C_Small
- added Ct1: 60p, symbol Device:C_Trim_Small
- added J1: DIP-16, Package_DIP:DIP-16_W7.62mm_Socket, symbol Connector_Generic:Conn_02x08_Odd_Even
- added Q10, Q11, Q12, Q2, Q3, Q4, Q5, Q6, Q7, Q8, Q9: Q_NJFET_DGS, symbol Device:Q_NJFET_DGS
- added R1: 10M, symbol Device:R_Small
- added R10, R11, R12, R13, R14, R4, R5, R6, R7, R8, R9: 10k, symbol Device:R_Small
- added R2: 4k7, symbol Device:R_Small
- added U1: 74HC04, symbol 74xx:74HC04
- added U10, U11, U12, U13, U3, U4, U5, U6, U7, U8, U9: ATtiny4-TS, Package_TO_SOT_SMD:SOT-23-6, symbol MCU_Microchip_ATtiny:ATtiny4-TS
- added U14: AZ1117-5.0, symbol Regulator_Linear:AZ1117-5.0
- added Y1: 2MHz, symbol Device:Crystal
- R3: renamed from R1; value R_Small -> 10k
- renumbered C4 to C6, U9 to U2
Connections:
- net +12V is gone; now on net +5V: Q1.2 (G), R3.1
- net GND: now also C1.1, C10.2, C11.2, C12.2, C13.2, C14.2, C15.2, C16.2, C17.2, C2.2, C3.2, C4.2, C5.2, C7.2, C8.2, C9.2, Ct1.2, J1.5 (Pin_5), U1.7 (GND), U10.2 (GND), U11.2 (GND), U12.2 (GND), U13.2 (GND), U14.1 (GND), U3.2 (GND), U4.2 (GND), U5.2 (GND), U6.2 (GND), U7.2 (GND), U8.2 (GND), U9.2 (GND)
- net VCC: now also C10.1, J1.1 (Pin_1), U14.3 (VI); no longer U2.5 (VCC)
- net +5V: now reaches C6.1
- net +5V: now also U2.5 (VCC), C11.1, C12.1, C13.1, C14.1, C15.1, C16.1, C17.1, C2.1, C4.1, C5.1, C7.1, C8.1, C9.1, Q10.2 (G), Q11.2 (G), Q12.2 (G), Q2.2 (G), Q3.2 (G), Q4.2 (G), Q5.2 (G), Q6.2 (G), Q7.2 (G), Q8.2 (G), Q9.2 (G), R10.1, R11.1, R12.1, R13.1, R14.1, R4.1, R5.1, R6.1, R7.1, R8.1, R9.1, U1.14 (VCC), U10.5 (VCC), U11.5 (VCC), U12.5 (VCC), U13.5 (VCC), U14.2 (VO), U3.5 (VCC), U4.5 (VCC), U5.5 (VCC), U6.5 (VCC), U7.5 (VCC), U8.5 (VCC), U9.5 (VCC)
- net CLK renamed CLK_A
- net CLK_A: now also U1.6, U3.3 (PB1), U4.3 (PB1)
- net DIVIDER_OUT renamed DIV_OUT_1
- net DIV_OUT_1: now also J1.2 (Pin_2)
- new net: Q2.3 (S), R4.2, U3.1 (PB0)
- new net: Q11.3 (S), R13.2, U12.1 (PB0)
- new net: Q7.3 (S), R9.2, U8.1 (PB0)
- new net: Q4.3 (S), R6.2, U5.1 (PB0)
- new net: Q9.3 (S), R11.2, U10.1 (PB0)
- new net: C1.2, Ct1.1, R1.1, U1.1, Y1.1
- new net: R1.2, R2.1, U1.2, U1.3
- new net: Q3.3 (S), R5.2, U4.1 (PB0)
- new net: Q5.3 (S), R7.2, U6.1 (PB0)
- new net: Q10.3 (S), R12.2, U11.1 (PB0)
- new net: Q8.3 (S), R10.2, U9.1 (PB0)
- new net: C3.1, R2.2, Y1.2
- new net: Q6.3 (S), R8.2, U7.1 (PB0)
- new net: Q12.3 (S), R14.2, U13.1 (PB0)
- new net CLK_B: U1.8, U5.3 (PB1), U6.3 (PB1), U7.3 (PB1)
- new net CLK_C: U1.10, U10.3 (PB1), U8.3 (PB1), U9.3 (PB1)
- new net CLK_D: U1.12, U11.3 (PB1), U12.3 (PB1), U13.3 (PB1)
- new net DIV_OUT_10: J1.10 (Pin_10), Q10.1 (D)
- new net DIV_OUT_11: J1.8 (Pin_8), Q11.1 (D)
- new net DIV_OUT_12: J1.6 (Pin_6), Q12.1 (D)
- new net DIV_OUT_2: J1.7 (Pin_7), Q2.1 (D)
- new net DIV_OUT_3: J1.9 (Pin_9), Q3.1 (D)
- new net DIV_OUT_4: J1.11 (Pin_11), Q4.1 (D)
- new net DIV_OUT_5: J1.13 (Pin_13), Q5.1 (D)
- new net DIV_OUT_6: J1.15 (Pin_15), Q6.1 (D)
- new net DIV_OUT_7: J1.16 (Pin_16), Q7.1 (D)
- new net DIV_OUT_8: J1.14 (Pin_14), Q8.1 (D)
- new net DIV_OUT_9: J1.12 (Pin_12), Q9.1 (D)
- new net M_CLK: U1.11, U1.13, U1.4, U1.5, U1.9
- no-connect marks 2 -> 26
Other:
- note added: "CLOCK DISTRIBUTION"
- note added: "MASTER CLOCK"
- note added: "Source : Elektor N°89 11/1985 - Page 11-52"
- moved on the sheet: C6, Q1, R3, U2

Commit message: Fix level shifter
Parts:
- removed Q1, Q10, Q11, Q12, Q2, Q3, Q4, Q5, Q6, Q7, Q8, Q9: Q_NJFET_DGS, symbol Device:Q_NJFET_DGS
- added Q1, Q10, Q11, Q12, Q2, Q3, Q4, Q5, Q6, Q7, Q8, Q9: Q_NMOS_GDS, symbol Device:Q_NMOS_GDS
- added R12, R13, R14, R15, R19, R20, R21, R25, R26, R27, R6, R7, R8: 10k, symbol Device:R_Small
- renumbered C11 to C10, C12 to C11, C13 to C12, C14 to C13, C15 to C14, C16 to C15, C10 to C16, R7 to R10, R8 to R11, R9 to R16, R10 to R17, R11 to R18, R12 to R22, R13 to R23, R14 to R24, R6 to R9, U9 to U10, U10 to U11, U11 to U12, U12 to U13, U13 to U14, U14 to U8, U8 to U9
Connections:
- net +5V: now also Q1.1 (G), Q10.1 (G), Q11.1 (G), Q12.1 (G), Q2.1 (G), Q3.1 (G), Q4.1 (G), Q5.1 (G), Q6.1 (G), Q7.1 (G), Q8.1 (G), Q9.1 (G)
- net DIV_OUT_1: now also Q1.2 (D), R6.2
- net DIV_OUT_10: now also Q10.2 (D), R25.2
- net DIV_OUT_11: now also Q11.2 (D), R26.2
- net DIV_OUT_12: now also Q12.2 (D), R27.2
- net DIV_OUT_2: now also Q2.2 (D), R7.2
- net DIV_OUT_3: now also Q3.2 (D), R8.2
- net DIV_OUT_4: now also Q4.2 (D), R12.2
- net DIV_OUT_5: now also Q5.2 (D), R13.2
- net DIV_OUT_6: now also Q6.2 (D), R14.2
- net DIV_OUT_7: now also Q7.2 (D), R19.2
- net DIV_OUT_8: now also Q8.2 (D), R20.2
- net DIV_OUT_9: now also Q9.2 (D), R21.2
- net VCC: now also R12.1, R13.1, R14.1, R15.1, R19.1, R20.1, R21.1, R25.1, R26.1, R27.1, R6.1, R7.1, R8.1
- net at R3.2, U2.1 (PB0): now also Q1.3 (S)
- net at R4.2, U3.1 (PB0): now also Q2.3 (S)
- net at R23.2, U13.1 (PB0): now also Q11.3 (S)
- net at R16.2, U9.1 (PB0): now also Q7.3 (S)
- net at R9.2, U5.1 (PB0): now also Q4.3 (S)
- net at R18.2, U11.1 (PB0): now also Q9.3 (S)
- net at R5.2, U4.1 (PB0): now also Q3.3 (S)
- net at R10.2, U6.1 (PB0): now also Q5.3 (S)
- net at R22.2, U12.1 (PB0): now also Q10.3 (S)
- net at R17.2, U10.1 (PB0): now also Q8.3 (S)
- net at R11.2, U7.1 (PB0): now also Q6.3 (S)
- net at R24.2, U14.1 (PB0): now also Q12.3 (S)

Commit message: Fix wrong header for MK50242
Parts:
- removed R15: 10k, symbol Device:R_Small
- removed U8: AZ1117-5.0, symbol Regulator_Linear:AZ1117-5.0
- added U8: uA7805, symbol Regulator_Linear:uA7805
- C16, C17: value 22u -> 10u
Connections:
- net +5V: now also U8.3 (OUT)
- net DIV_OUT_1: now also J1.16 (Pin_16); no longer J1.2 (Pin_2)
- net DIV_OUT_10: now also J1.11 (Pin_11); no longer J1.10 (Pin_10)
- net DIV_OUT_11: now also J1.7 (Pin_7); no longer J1.8 (Pin_8)
- net DIV_OUT_12: now also J1.8 (Pin_8); no longer J1.6 (Pin_6)
- net DIV_OUT_2: now also J1.3 (Pin_3); no longer J1.7 (Pin_7)
- net DIV_OUT_3: now also J1.15 (Pin_15); no longer J1.9 (Pin_9)
- net DIV_OUT_4: now also J1.4 (Pin_4); no longer J1.11 (Pin_11)
- net DIV_OUT_5: now also J1.14 (Pin_14); no longer J1.13 (Pin_13)
- net DIV_OUT_6: now also J1.13 (Pin_13); no longer J1.15 (Pin_15)
- net DIV_OUT_7: now also J1.5 (Pin_5); no longer J1.16 (Pin_16)
- net DIV_OUT_8: now also J1.6 (Pin_6); no longer J1.14 (Pin_14)
- net GND: now also J1.10 (Pin_10), U1.3, U8.2 (GND); no longer J1.5 (Pin_5)
- net M_CLK: now also R1.2, R2.1, U1.2; no longer U1.4
- net VCC: now also U8.1 (IN)
- no-connect marks 26 -> 27
Other:
- note added: "DIP HEADER"
- note added: "DIVIDERS"
- note added: "PSU"
- moved on the sheet: C10, C11, C12, C13, C14, C15, C16, C17, C2, C4, C5, C6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

Commit message: Replace all mosfet by 2 cd4504
Parts:
- removed Q1, Q10, Q11, Q12, Q2, Q3, Q4, Q5, Q6, Q7, Q8, Q9: Q_NMOS_GDS, symbol Device:Q_NMOS_GDS
- removed R10, R11, R12, R13, R14, R16, R17, R18, R19, R20, R21, R22, R23, R24, R25, R26, R27, R3, R4, R5, R6, R7, R8, R9: 10k, symbol Device:R_Small
- added C16, C17, C18, C19, C22, C23: 100n, Resistor_SMD:R_0805_2012Metric_Pad1.20x1.40mm_HandSolder, symbol Device:C_Small
- added U11, U6: 4504, Package_SO:SO-16_3.9x9.9mm_P1.27mm, symbol 4xxx_IEEE:4504
- C1: footprint (none) -> Capacitor_SMD:C_1206_3216Metric
- C10, C11, C12, C13, C14, C15, C4, C5, C6, C7, C8, C9: footprint Capacitor_SMD:C_1206_3216Metric_Pad1.42x1.75mm_HandSolder -> Resistor_SMD:R_0805_2012Metric_Pad1.20x1.40mm_HandSolder
- C2: renamed from C3; footprint (none) -> Capacitor_SMD:C_1206_3216Metric
- C3: renamed from C2; footprint Capacitor_SMD:C_1206_3216Metric_Pad1.42x1.75mm_HandSolder -> Resistor_SMD:R_0805_2012Metric_Pad1.20x1.40mm_HandSolder
- R1, R2: footprint (none) -> Resistor_SMD:R_0805_2012Metric_Pad1.20x1.40mm_HandSolder
- U1: footprint (none) -> Package_SO:SOIC-14_3.9x8.7mm_P1.27mm
- U16: renamed from U8; footprint (none) -> Package_TO_SOT_SMD:SOT-223
- Y1: footprint (none) -> Package_TO_SOT_SMD:SOT-89-5
- renumbered C17 to C20, C16 to C21, U13 to U10, U4 to U12, U7 to U13, U11 to U14, U14 to U15, U5 to U3, U9 to U4, U12 to U5, U3 to U7, U6 to U8, U10 to U9
Connections:
- net +5V: now also C16.1, C17.1, C18.1, C19.1, U11.1 (Vcc), U11.13 (EN), U6.1 (Vcc), U6.13 (EN)
- net DIV_OUT_1: now also U11.2
- net DIV_OUT_10: now also U11.15
- net DIV_OUT_11: now also U6.12
- net DIV_OUT_12: now also U6.15
- net DIV_OUT_2: now also U6.2
- net DIV_OUT_3: now also U11.4
- net DIV_OUT_4: now also U6.4
- net DIV_OUT_5: now also U11.6
- net DIV_OUT_6: now also U11.10
- net DIV_OUT_7: now also U6.6
- net DIV_OUT_8: now also U6.10
- net DIV_OUT_9: now also U11.12
- net GND: now also C16.2, C17.2, C18.2, C19.2
- net VCC: now also U11.16 (Vdd), U6.16 (Vdd)
- net OUT_1: now reaches U2.1 (PB0)
- net OUT_1: now also U11.3
- net OUT_2: now reaches U7.1 (PB0)
- net OUT_2: now also U6.3
- net OUT_11: now reaches U10.1 (PB0)
- net OUT_11: now also U6.11
- net OUT_7: now reaches U4.1 (PB0)
- net OUT_7: now also U6.7
- net OUT_10: now reaches U5.1 (PB0)
- net OUT_10: now also U11.14
- net OUT_9: now reaches U14.1 (PB0)
- net OUT_9: now also U11.11
- net OUT_3: now reaches U12.1 (PB0)
- net OUT_3: now also U11.5
- net OUT_5: now reaches U8.1 (PB0)
- net OUT_5: now also U11.7
- net OUT_8: now reaches U9.1 (PB0)
- net OUT_8: now also U6.9
- net OUT_6: now reaches U13.1 (PB0)
- net OUT_6: now also U11.9
- net OUT_4: now reaches U3.1 (PB0)
- net OUT_4: now also U6.5
- net OUT_12: now reaches U15.1 (PB0)
- net OUT_12: now also U6.14
- new net: C22.1, C23.1
- new net: C22.2, C23.2
Other:
- note added: "Adjust Ct1 to 2.00024MHz"
- moved on the sheet: C1, C10, C11, C12, C13, C14, C15, C2, C20, C21, C3, C4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
